Commit message: addition of new end-effector type franka_hand_with_camera that accounts for the new camera support

File: robots/common/franka_robot.xacro (robot description, xacro)
@@ -95,4 +95,34 @@
       />
     </xacro:if>
+    <xacro:if value="${hand and ee_id == 'franka_hand_with_camera'}">
+      <xacro:include filename="$(find franka_description)/end_effectors/common/utils.xacro" />
+      <xacro:include filename="$(find franka_description)/end_effectors/$(arg ee_id)/$(arg ee_id).urdf.xacro" />
+      <xacro:include filename="$(find franka_description)/end_effectors/$(arg ee_id)/$(arg ee_id)_arguments.xacro" />
+      <xacro:if value="${arm_id == 'fp3'}">
+        <xacro:property name="ee_color" value="black" />
+      </xacro:if>
+      <xacro:if value="${arm_id == 'fr3' or arm_id == 'fer'}">
+        <xacro:property name="ee_color" value="white" />
+      </xacro:if>
+      <xacro:property name="special_connection" value="$(arg special_connection)" />
+      <xacro:property name="default_connection" value="${(arm_id + '_link8') if not use_ft_sensor else 'ati_mini45_tool_mount'}" />
+      <xacro:property name="connection" value="${special_connection if special_connection != '' else default_connection}" />
+      <xacro:franka_hand_with_camera
+        connected_to="${arm_prefix_modified}${connection}"
+        arm_id="${arm_id}"
+        arm_prefix="${arm_prefix_modified}"
+        ee_id="${ee_id}_${ee_color}"
+        ee_inertials="${xacro.load_yaml('$(find franka_description)/end_effectors/$(arg ee_id)/inertials.yaml')}"
+        rpy_ee="$(arg rpy_ee)"
+        xyz_ee="$(arg xyz_ee)"
+        tcp_xyz="$(arg tcp_xyz)"
+        tcp_rpy="$(arg tcp_rpy)"
+        hand_mesh_id="franka_hand_${ee_color}"
+        safety_distance="$(arg safety_distance)"
+        gazebo="${gazebo}"
+        description_pkg="$(arg description_pkg)"
+        with_sc="${with_sc}"
+      />
+    </xacro:if>
     <xacro:if value="${hand and ee_id == 'ati_mini45_with_camera'}">
       <xacro:include filename="$(find franka_description)/end_effectors/common/utils.xacro" />
@@ -133,5 +163,5 @@
           with_sc="${with_sc}" />
     </xacro:if>
-    <xacro:if value="${hand and ee_id != 'none' and ee_id != 'franka_hand' and ee_id != 'ati_mini45_with_camera' and ee_id != 'ati_mini45_no_camera'}">
+    <xacro:if value="${hand and ee_id != 'none' and ee_id != 'franka_hand' and ee_id != 'franka_hand_with_camera' and ee_id != 'ati_mini45_with_camera' and ee_id != 'ati_mini45_no_camera'}">
       <xacro:include filename="$(find franka_description)/end_effectors/common/ee_with_one_link.xacro"/>
       <xacro:include filename="$(find franka_description)/end_effectors/common/utils.xacro" />
@@ -178,5 +208,5 @@
       </xacro:sensor_d435>
       <!-- camera support -->
-      <xacro:unless value="${ee_id == 'ati_mini45_with_camera'}">
+      <xacro:unless value="${ee_id == 'ati_mini45_with_camera' or ee_id == 'franka_hand_with_camera'}">
         <link name="${arm_id}_camera_support_link">
           <inertial>
@@ -247,5 +277,5 @@
          tip="${arm_id}_joint8"
        />
-      <xacro:if value="${ee_id == 'franka_hand'}">
+      <xacro:if value="${ee_id == 'franka_hand' or ee_id == 'franka_hand_with_camera'}">
         <xacro:gazebo-joint joint="${arm_id}_finger_joint1" transmission="hardware_interface/EffortJointInterface" />
         <xacro:gazebo-joint joint="${arm_id}_finger_joint2" transmission="hardware_interface/EffortJointInterface" />
