Commit message: Adjust visuals still need to provide the camera calib parameters in the right frame

File: end_effectors/common/franka_hand.xacro (robot description, xacro)
@@ -2,5 +2,5 @@
 <robot xmlns:xacro="http://www.ros.org/wiki/xacro" name="hand">
   <!-- safety_distance: Minimum safety distance in [m] by which the collision volumes are expanded and which is enforced during robot motions -->
-  <xacro:macro name="franka_hand" params="connected_to:='' arm_id arm_prefix:='' ee_id ee_inertials rpy_ee:='0 0 0' xyz_ee:='0 0 0' tcp_xyz:='0 0 0.1034' tcp_rpy:='0 0 0' safety_distance:=0 gazebo:=false description_pkg:=franka_description with_sc:=false">
+  <xacro:macro name="franka_hand" params="connected_to:='' arm_id arm_prefix:='' ee_id ee_inertials rpy_ee:='0 0 0' xyz_ee:='0 0 0' tcp_xyz:='0 0 0.1034' tcp_rpy:='0 0 0' safety_distance:=0 gazebo:=false description_pkg:=franka_description with_sc:=false mesh_offset_xyz:='0 0 0' mesh_offset_rpy:='0 0 0'">
     <xacro:property name="ee_prefix" default="robot_"/>
     <xacro:unless value="${arm_id == ''}">
@@ -14,5 +14,13 @@
       </joint>
     </xacro:unless>
-    <xacro:ee_link_with_sc name="hand" gazebo="${gazebo}" with_sc="${with_sc}">
+    <xacro:property name="finger_visual_rpy_right"
+                    value="${mesh_offset_rpy.split(' ')[0]} ${mesh_offset_rpy.split(' ')[1]} ${float(mesh_offset_rpy.split(' ')[2]) + pi}" />
+    <xacro:ee_link_with_sc name="hand"
+                           gazebo="${gazebo}"
+                           with_sc="${with_sc}"
+                           visual_xyz="${mesh_offset_xyz}"
+                           visual_rpy="${mesh_offset_rpy}"
+                           collision_xyz="${mesh_offset_xyz}"
+                           collision_rpy="${mesh_offset_rpy}">
       <self_collision_geometries>
         <xacro:collision_capsule xyz="0 0 0.04" direction="y" radius="${0.04+safety_distance}" length="0.1" />
@@ -29,4 +37,5 @@
     <link name="${ee_prefix}leftfinger">
       <visual name="${ee_prefix}leftfinger_visual">
+        <origin xyz="${mesh_offset_xyz}" rpy="${mesh_offset_rpy}" />
         <geometry>
           <mesh filename="package://${description_pkg}/meshes/robot_ee/${ee_id}/visual/finger.dae" />
@@ -67,5 +76,5 @@
     <link name="${ee_prefix}rightfinger">
       <visual name="${ee_prefix}rightfinger_visual">
-        <origin xyz="0 0 0" rpy="0 0 ${pi}" />
+        <origin xyz="${mesh_offset_xyz}" rpy="${finger_visual_rpy_right}" />
         <geometry>
           <mesh filename="package://${description_pkg}/meshes/robot_ee/${ee_id}/visual/finger.dae" />

File: end_effectors/common/utils.xacro (robot description, xacro)
@@ -32,8 +32,9 @@
   <!-- self_collision_geometries:  self <collision> models        -->
   <!-- ========================================================== -->
-  <xacro:macro name="ee_link_with_sc" params="name prefix=${ee_prefix} rpy:='0 0 0' **self_collision_geometries gazebo:=false with_sc:=false">
+  <xacro:macro name="ee_link_with_sc" params="name prefix=${ee_prefix} rpy:='0 0 0' visual_xyz:='0 0 0' visual_rpy:='0 0 0' collision_xyz:='0 0 0' collision_rpy:='0 0 0' **self_collision_geometries gazebo:=false with_sc:=false">
     <!-- sub-link defining detailed meshes for collision with environment -->
     <link name="${prefix}${name}">
       <visual name="${prefix}${name}_visual">
+        <origin xyz="${visual_xyz}" rpy="${visual_rpy}" />
         <geometry>
           <mesh filename="package://${description_pkg}/meshes/robot_ee/${ee_id}/visual/${name}.dae" />
@@ -41,4 +42,5 @@
       </visual>
       <collision name="${prefix}${name}_collision">
+        <origin xyz="${collision_xyz}" rpy="${collision_rpy}" />
         <geometry>
           <mesh filename="package://franka_description/meshes/robot_ee/${ee_id}/collision/${name}.stl" />

File: end_effectors/franka_hand_with_camera/franka_hand_with_camera.urdf.xacro (robot description, xacro)
@@ -11,6 +11,8 @@
     <xacro:property name="camera_support_offset_xyz" value="0 0 0" />
     <xacro:property name="camera_support_offset_rpy" value="0 0 0" />
-    <xacro:property name="hand_offset_xyz" value="0 0 0.1" />
-    <xacro:property name="hand_offset_rpy" value="0 0 0.1" />
+    <xacro:property name="hand_offset_xyz" value="0 0 0.0065" />
+    <xacro:property name="hand_offset_rpy" value="0 0 0" />
+    <xacro:property name="mesh_offset_xyz" value="0 0 0" />
+    <xacro:property name="mesh_offset_rpy" value="0 0 -${pi / 4}" />
     <xacro:unless value="${connected_to == ''}">
       <joint name="${ee_prefix}camera_support_joint" type="fixed">
@@ -27,5 +29,5 @@
       </inertial>
       <visual>
-        <origin xyz="0.022 0 -0.012" rpy="${pi} 0 -${pi / 2}"/>
+        <origin xyz="0.0 0 0.0035" rpy="0 0 -${pi / 4}"/>
         <geometry>
           <mesh filename="package://franka_description/meshes/robot_ee/franka_hand_with_camera/camera_support.stl" />
@@ -36,5 +38,5 @@
       </visual>
       <collision>
-        <origin xyz="0.022 0 -0.012" rpy="${pi} 0 -${pi / 2}"/>
+        <origin xyz="0.0 0 0.0035" rpy="0 0 -${pi / 4}"/>
         <geometry>
           <mesh filename="package://franka_description/meshes/robot_ee/franka_hand_with_camera/camera_support.stl" />
@@ -49,4 +51,6 @@
                        rpy_ee="${hand_offset_rpy}"
                        xyz_ee="${hand_offset_xyz}"
+                       mesh_offset_xyz="${mesh_offset_xyz}"
+                       mesh_offset_rpy="${mesh_offset_rpy}"
                        tcp_xyz="${tcp_xyz}"
                        tcp_rpy="${tcp_rpy}"
