Commit message: fix wrong orientation of the hand for end effector franka hand with cam

File: end_effectors/franka_hand_with_camera/franka_hand_with_camera.urdf.xacro (robot description, xacro)
@@ -12,7 +12,7 @@
     <xacro:property name="camera_support_offset_rpy" value="0 0 0" />
     <xacro:property name="hand_offset_xyz" value="0 0 0.0065" />
-    <xacro:property name="hand_offset_rpy" value="0 0 0" />
+    <xacro:property name="hand_offset_rpy" value="0 0 -0.7853981633974483" />
     <xacro:property name="mesh_offset_xyz" value="0 0 0" />
-    <xacro:property name="mesh_offset_rpy" value="0 0 -${pi / 4}" />
+    <xacro:property name="mesh_offset_rpy" value="0 0 0" />
     <xacro:unless value="${connected_to == ''}">
       <joint name="${ee_prefix}camera_support_joint" type="fixed">

File: robots/common/franka_robot.xacro (robot description, xacro)
@@ -204,5 +204,5 @@
       <!-- use_mesh="true" produces an error when visualizing with rviz2
       because the generated urdf contains mesh filename paths that do not start with file:// -->
-      <xacro:sensor_d435 parent="${arm_id}_ref_camera_link" name="camera" use_nominal_extrinsics="false" use_mesh="true">
+      <xacro:sensor_d435 parent="${arm_id}_ref_camera_link" name="camera" use_nominal_extrinsics="true" use_mesh="true">
         <origin xyz="0 0 0" rpy="0 0 0"/>
       </xacro:sensor_d435>
